File: pcb/qez.sch (KiCad schematic (older format))
At the start: 79 parts, among them U1 ATmega32U2-AU, U2 SRV05-4, X1 Crystal_GND24_Small

Commit message: Update qez.sch
Parts:
- U1: LCSC (none) -> C618733
Changed lines of the file:
@@
 F 2 "Package_QFP:TQFP-32_7x7mm_P0.8mm" H 3400 2750 50  0001 C CIN
 F 3 "http://ww1.microchip.com/downloads/en/DeviceDoc/doc7799.pdf" H 3400 2750 50  0001 C CNN
+F 4 "C618733" H 3400 2750 50  0001 C CNN "LCSC"
 	1    3400 2750
 	1    0    0    -1
